Commit message: Collision geometry added for R2D2.urdf robot

File: demos/models/robots/R2D2.urdf (robot description, URDF)
Before this commit: robot R2D2, 12 links, 11 joints
Links:
- link base_link: geometry collision box size=0.4 0.4 0.6; visual cylinder length=0.6 radius=0.2
- link gripper_pole: geometry collision box size=0.02 0.02 0.2; visual cylinder length=0.2 radius=.01
- link head: geometry collision box size=0.4 0.4 0.4; visual sphere radius=0.2
- link left_back_wheel: geometry collision box size=0.07 0.07 0.1; visual cylinder length=.1 radius=0.035
- link left_front_wheel: geometry collision box size=0.07 0.07 0.1; visual cylinder length=.1 radius=0.035
- link right_back_wheel: geometry collision box size=0.07 0.07 0.1; visual cylinder length=.1 radius=0.035
- link right_front_wheel: geometry collision box size=0.07 0.07 0.1; visual cylinder length=.1 radius=0.035
