Commit message: Solved problems in baxter collision model

File: demos/models/robots/baxter.urdf (robot description, URDF)
Before this commit: robot baxter, 28 links, 27 joints
Links:
- link left_lower_shoulder: geometry collision cylinder length=0.107 radius=0.06; collision cylinder length=0.12 radius=0.06
- link left_upper_elbow: geometry collision cylinder length=0.273 radius=0.06; visual mesh filename=baxter/upper_elbow/E0.wrl scale=1000 1000 1000
- link right_lower_shoulder: geometry collision cylinder length=0.107 radius=0.06; collision cylinder length=0.12 radius=0.06
- link right_upper_elbow: geometry collision cylinder length=0.273 radius=0.06; visual mesh filename=baxter/upper_elbow/E0.wrl scale=1000 1000 1000
