Commit message: Updated urdf robots

File: demos/models/robots/AllegroHandR.urdf (robot description, URDF)
Before this commit: robot allegro_hand_right, 21 links, 20 joints
Links:
- link link_11_0_tip: geometry collision box size=0.019 0.023 0.0365; visual mesh filename=AllegroHand/right/sensing_tip.wrl
- link link_15_0_tip: geometry collision box size=0.019 0.023 0.0365; visual mesh filename=AllegroHand/right/sensing_tip.wrl
- link link_3_0_tip: geometry collision box size=0.019 0.023 0.0365; visual mesh filename=AllegroHand/right/sensing_tip.wrl
- link link_7_0_tip: geometry collision box size=0.019 0.023 0.0365; visual mesh filename=AllegroHand/right/sensing_tip.wrl
Joints:
- joint joint_11_0_tip: origin xyz=0 0 0.0267 rpy=0 0 0 -> xyz=0 0 0.0267
- joint joint_15_0_tip: origin xyz=0 0 0.0423 rpy=0 0 0 -> xyz=0 0 0.0423
- joint joint_3_0_tip: origin xyz=0 0 0.0267 rpy=0 0 0 -> xyz=0 0 0.0267
- joint joint_7_0_tip: origin xyz=0 0 0.0267 rpy=0 0 0 -> xyz=0 0 0.0267

File: demos/models/robots/R2D2.urdf (robot description, URDF)
Before this commit: robot R2D2, 12 links, 11 joints
Links:
- link base_link: geometry visual cylinder length=0.6 radius=0.2
- link gripper_pole: geometry visual cylinder length=0.2 radius=.01
- link head: geometry visual sphere radius=0.2
- link left_back_wheel: geometry visual cylinder length=.1 radius=0.035
- link left_front_wheel: geometry visual cylinder length=.1 radius=0.035
- link right_back_wheel: geometry visual cylinder length=.1 radius=0.035
- link right_front_wheel: geometry visual cylinder length=.1 radius=0.035
Joints:
- joint gripper_extension: limit (none) -> lower=-0.38 upper=0 effort=1000.0 velocity=0.5; type fixed -> prismatic
- joint head_swivel: axis (none) -> 0 0 1; limit (none) -> lower=-3.1415 upper=3.1415; type fixed -> revolute
- joint left_back_wheel_joint: axis (none) -> 0 0 1; limit (none) -> lower=-3.1415 upper=3.1415 effort=100 velocity=100; type fixed -> revolute
- joint left_front_wheel_joint: axis (none) -> 0 0 1; limit (none) -> lower=-3.1415 upper=3.1415 effort=100 velocity=100; type fixed -> revolute
- joint right_back_wheel_joint: axis (none) -> 0 0 1; limit (none) -> lower=-3.1415 upper=3.1415 effort=100 velocity=100; type fixed -> revolute
- joint right_front_wheel_joint: axis (none) -> 0 0 1; limit (none) -> lower=-3.1415 upper=3.1415 effort=100 velocity=100; type fixed -> revolute

Commit message: Updated demos

File: demos/models/robots/AllegroHandR.urdf (robot description, URDF)
Before this commit: robot allegro_hand_right, 21 links, 20 joints
Links:
- removed link Palm
- added link base_link; collision box size=0.0408 0.1130 0.095; visual mesh filename=AllegroHand/right/base_link_right.wrl scale=0.001 0.001 0.001
Joints:
- joint joint_0.0: parent Palm -> base_link
- joint joint_12.0: parent Palm -> base_link
- joint joint_4.0: parent Palm -> base_link
- joint joint_8.0: parent Palm -> base_link
