Commit message: Updated demos

File: demos/models/robots/AllegroHandL.urdf (robot description, URDF)
Before this commit: robot allegro_hand_left, 21 links, 20 joints
Links:
- link base_link: geometry collision box size=0.0408 0.1130 0.095; visual mesh filename=AllegroHand/left/base_link_left.wrl scale=0.001 0.001 0.001
- link link_0.0: geometry collision box size=0.0196 0.0275 0.0164; visual mesh filename=AllegroHand/left/link_0_0.wrl scale=0.001 0.001 0.001
- link link_1.0: geometry collision box size=0.0196 0.0275 0.054; visual mesh filename=AllegroHand/left/link_1_0.wrl scale=0.001 0.001 0.001
- link link_10.0: geometry collision box size=0.0196 0.0275 0.0384; visual mesh filename=AllegroHand/left/link_2_0.wrl scale=0.001 0.001 0.001
- link link_11.0: geometry collision box size=0.0196 0.0275 0.0267; visual mesh filename=AllegroHand/left/link_3_0.wrl scale=0.001 0.001 0.001
- link link_11.0_tip: geometry collision box size=0.019 0.023 0.0365; visual mesh filename=AllegroHand/left/sensing_tip.wrl scale=0.001 0.001 0.001
- link link_12.0: geometry collision box size=0.0358 0.034 0.0455; visual mesh filename=AllegroHand/left/link_12_0_left.wrl scale=0.001 0.001 0.001
- link link_13.0: geometry collision box size=0.0196 0.0275 0.0177; visual mesh filename=AllegroHand/left/link_13_0.wrl scale=0.001 0.001 0.001
- link link_14.0: geometry collision box size=0.0196 0.0275 0.0514; visual mesh filename=AllegroHand/left/link_14_0.wrl scale=0.001 0.001 0.001
- link link_15.0: geometry collision box size=0.0196 0.0275 0.0423; visual mesh filename=AllegroHand/left/link_15_0.wrl scale=0.001 0.001 0.001
- link link_15.0_tip: geometry collision sphere radius=0.012; visual mesh filename=AllegroHand/right/link_3_0_tip.wrl scale=0.001 0.001 0.001
- link link_2.0: geometry collision box size=0.0196 0.0275 0.0384; visual mesh filename=AllegroHand/left/link_2_0.wrl scale=0.001 0.001 0.001
- link link_3.0: geometry collision box size=0.0196 0.0275 0.0267; visual mesh filename=AllegroHand/left/link_3_0.wrl scale=0.001 0.001 0.001
- link link_3.0_tip: geometry collision sphere radius=0.012; visual mesh filename=AllegroHand/right/link_3_0_tip.wrl scale=0.001 0.001 0.001
- link link_4.0: geometry collision box size=0.0196 0.0275 0.0164; visual mesh filename=AllegroHand/left/link_0_0.wrl scale=0.001 0.001 0.001
- link link_5.0: geometry collision box size=0.0196 0.0275 0.054; visual mesh filename=AllegroHand/left/link_1_0.wrl scale=0.001 0.001 0.001
- link link_6.0: geometry collision box size=0.0196 0.0275 0.0384; visual mesh filename=AllegroHand/left/link_2_0.wrl scale=0.001 0.001 0.001
- link link_7.0: geometry collision box size=0.0196 0.0275 0.0267; visual mesh filename=AllegroHand/left/link_3_0.wrl scale=0.001 0.001 0.001
- link link_7.0_tip: geometry collision sphere radius=0.012; visual mesh filename=AllegroHand/right/link_3_0_tip.wrl scale=0.001 0.001 0.001
- link link_8.0: geometry collision box size=0.0196 0.0275 0.0164; visual mesh filename=AllegroHand/left/link_0_0.wrl scale=0.001 0.001 0.001
- link link_9.0: geometry collision box size=0.0196 0.0275 0.054; visual mesh filename=AllegroHand/left/link_1_0.wrl scale=0.001 0.001 0.001
Joints:
- joint joint_11.0_tip: origin xyz=0 0 0.0267 rpy=0 0 0 -> xyz=0 0 0.0267
- joint joint_12.0: axis +1 0 0 -> 1 0 0
- joint joint_15.0_tip: origin xyz=0 0 0.0423 rpy=0 0 0 -> xyz=0 0 0.0423
- joint joint_3.0_tip: origin xyz=0 0 0.0267 rpy=0 0 0 -> xyz=0 0 0.0267
- joint joint_4.0: origin xyz=0 0 0.0007 rpy=0.0 0 0 -> xyz=0 0 0.0007
- joint joint_7.0_tip: origin xyz=0 0 0.0267 rpy=0 0 0 -> xyz=0 0 0.0267
