Commit message: Updated demos

File: demos/models/robots/UR5_AllegroHandL.urdf (robot description, URDF)
Before this commit: robot UR5_AllegroHandL, 29 links, 28 joints
Links:
- link Palm: geometry collision box size=0.0408 0.1130 0.095; visual mesh filename=AllegroHand/left/base_link_left.wrl scale=0.001 0.001 0.001

Commit message: Updated demos

File: demos/models/robots/UR5_AllegroHandL.urdf (robot description, URDF)
Before this commit: robot UR5_AllegroHandL, 29 links, 28 joints
Links:
- link Support: geometry collision cylinder length=0.043 radius=0.0355; visual mesh filename=UR5/AH_support.wrl scale=0.001 0.001 0.001
- link link_11_0_tip: geometry collision box size=0.019 0.023 0.025; collision cylinder length=0.019 radius=0.0115
- link link_15_0_tip: geometry collision box size=0.019 0.023 0.025; collision cylinder length=0.019 radius=0.0115
- link link_3_0_tip: geometry collision box size=0.019 0.023 0.025; collision cylinder length=0.019 radius=0.0115
- link link_7_0_tip: geometry collision box size=0.019 0.023 0.025; collision cylinder length=0.019 radius=0.0115
Joints:
- joint SupportJoint: origin xyz=0 0.0983 0 rpy=-1.570796325 0 0 -> xyz=0 0.1089 0 rpy=-1.570796325 0 0

File: demos/models/robots/UR5_AllegroHandR.urdf (robot description, URDF)
Before this commit: robot UR5_AllegroHandR, 29 links, 28 joints
Links:
- link Support: geometry collision cylinder length=0.043 radius=0.0355; visual mesh filename=UR5/AH_support.wrl scale=0.001 0.001 0.001
- link link_11_0_tip: geometry collision box size=0.019 0.023 0.025; collision cylinder length=0.019 radius=0.0115
- link link_15_0_tip: geometry collision box size=0.019 0.023 0.025; collision cylinder length=0.019 radius=0.0115
- link link_3_0_tip: geometry collision box size=0.019 0.023 0.025; collision cylinder length=0.019 radius=0.0115
- link link_7_0_tip: geometry collision box size=0.019 0.023 0.025; collision cylinder length=0.019 radius=0.0115
Joints:
- joint PalmJoint: origin xyz=0.009 0 0.111 rpy=0 0 1.570796327 -> xyz=0 0.009 0.111 rpy=0 0 1.570796327
- joint SupportJoint: origin xyz=0 0.0983 0 rpy=-1.570796325 0 0 -> xyz=0 0.1089 0 rpy=-1.570796325 0 0
