Commit message: Solved error in collision model

File: demos/models/robots/UR5_AllegroHandL_cylinder.urdf (robot description, URDF)
Before this commit: robot UR5_AllegroHandL, 30 links, 29 joints
Links:
- link Palm: geometry collision box size=0.0408 0.0965 0.095; collision box size=0.0408 0.113 0.0475

File: demos/models/robots/UR5_AllegroHandR_cylinder.urdf (robot description, URDF)
Before this commit: robot UR5_AllegroHandR, 30 links, 29 joints
Links:
- link Palm: geometry collision box size=0.0408 0.0965 0.095; collision box size=0.0408 0.113 0.0475

File: demos/models/robots/UR5_AllegroHandR_water.urdf (robot description, URDF)
Before this commit: robot UR5_AllegroHandR, 30 links, 29 joints
Links:
- link Palm: geometry collision box size=0.0408 0.0965 0.095; collision box size=0.0408 0.113 0.0475
