Commit message: added robotiq ttol to chess example

File: demos/models/robots/ur3_robotniq.urdf (robot description, URDF)
Before this commit: robot ur3_robotniq, 7 links, 6 joints
Links:
- added link coupler_link; collision cylinder length=0.0139 radius=0.0375; visual cylinder length=0.0139 radius=0.0375
- added link ee_link; collision box size=0.01 0.01 0.01; visual box size=0.01 0.01 0.01
- added link gripper_base; collision box size=0.03 0.04 0.06; collision cylinder length=0.045 radius=0.04
- added link gripper_left_coupler; collision box size=0.03 0.065 0.02; visual mesh filename=robotiq/visual/coupler.dae scale=0.001 0.001 0.001
- added link gripper_left_driver; collision box size=0.02 0.04 0.02; visual mesh filename=robotiq/visual/driver.dae scale=0.001 0.001 0.001
- added link gripper_left_follower; collision box size=0.02 0.015 0.048; visual mesh filename=robotiq/visual/follower.dae scale=0.001 0.001 0.001
- added link gripper_left_pad; collision box size=0.02 0.008 0.036; visual mesh filename=robotiq/visual/pad.dae scale=0.001 0.001 0.001
- added link gripper_left_spring_link; collision box size=0.04 0.02 0.065; visual mesh filename=robotiq/visual/spring_link.dae scale=0.001 0.001 0.001
- added link gripper_right_coupler; collision box size=0.03 0.065 0.02; visual mesh filename=robotiq/visual/coupler.dae scale=0.001 0.001 0.001
- added link gripper_right_driver; collision box size=0.02 0.04 0.02; visual mesh filename=robotiq/visual/driver.dae scale=0.001 0.001 0.001
- added link gripper_right_follower; collision box size=0.02 0.015 0.048; visual mesh filename=robotiq/visual/follower.dae scale=0.001 0.001 0.001
- added link gripper_right_pad; collision box size=0.02 0.008 0.036; visual mesh filename=robotiq/visual/pad.dae scale=0.001 0.001 0.001
- added link gripper_right_spring_link; collision box size=0.04 0.02 0.065; visual mesh filename=robotiq/visual/spring_link.dae scale=0.001 0.001 0.001
- added link tool0; collision box size=0.01 0.01 0.01; visual box size=0.01 0.01 0.01
Joints:
- added joint coupler_joint: type fixed, parent tool0, child coupler_link, origin xyz=0.0 0.0 0.0 rpy=0.0 0.0 0.0
- added joint coupler_link_gripper_base_joint: type fixed, parent coupler_link, child gripper_base, origin xyz=0 0 0.0079 rpy=0 0 1.57079632679
- added joint ee_fixed_joint: type fixed, parent wrist_3_link, child ee_link, origin xyz=0.0 0.0819 0.0 rpy=0.0 0.0 1.57079632679
- added joint gripper_left_coupler_joint: type fixed, parent gripper_left_driver, child gripper_left_coupler, origin xyz=0 0.0315 -0.0041 rpy=0 0 0
- added joint gripper_left_driver_joint: type revolute, parent gripper_base, child gripper_left_driver, origin xyz=0 -0.0306011 0.054904 rpy=0 0 3.141592653589793, axis 1 0 0, limit lower=0.0 upper=0.715584844444 effort=176 velocity=1.91986177778, mimic joint=gripper_right_driver_joint multiplier=1
- added joint gripper_left_follower_joint: type revolute, parent gripper_left_coupler, child gripper_left_follower, origin xyz=0 0.0061 0.0471 rpy=0 0 0, axis 1 0 0, limit lower=-2.96705911111 upper=2.96705911111 effort=176 velocity=1.91986177778, mimic joint=gripper_right_driver_joint multiplier=-1
- added joint gripper_left_pad_joint: type fixed, parent gripper_left_follower, child gripper_left_pad
- added joint gripper_left_spring_link_joint: type revolute, parent gripper_base, child gripper_left_spring_link, origin xyz=0 -0.012 0.0614 rpy=0 0 3.141592653589793, axis 1 0 0, limit lower=-2.96705911111 upper=2.96705911111 effort=176 velocity=1.91986177778, mimic joint=gripper_right_driver_joint multiplier=1
- added joint gripper_right_coupler_joint: type fixed, parent gripper_right_driver, child gripper_right_coupler, origin xyz=0 0.0315 -0.0041 rpy=0 0 0
- added joint gripper_right_driver_joint: type revolute, parent gripper_base, child gripper_right_driver, origin xyz=0 0.0306011 0.054904 rpy=0 0 0, axis 1 0 0, limit lower=0.0 upper=0.872664444444 effort=60 velocity=1.91986177778
- added joint gripper_right_follower_joint: type revolute, parent gripper_right_coupler, child gripper_right_follower, origin xyz=0 0.0061 0.0471 rpy=0 0 0, axis 1 0 0, limit lower=-2.96705911111 upper=2.96705911111 effort=176 velocity=1.91986177778, mimic joint=gripper_right_driver_joint multiplier=-1
- added joint gripper_right_pad_joint: type fixed, parent gripper_right_follower, child gripper_right_pad
- added joint gripper_right_spring_link_joint: type revolute, parent gripper_base, child gripper_right_spring_link, origin xyz=0 0.012 0.0614 rpy=0 0 0, axis 1 0 0, limit lower=-2.96705911111 upper=2.96705911111 effort=176 velocity=1.91986177778, mimic joint=gripper_right_driver_joint multiplier=1
- added joint wrist_3_link-tool0_fixed_joint: type fixed, parent wrist_3_link, child tool0, origin xyz=0 0.0819 0 rpy=-1.57079632679 0 0

Commit message: corrected robotniq gripper movement in chess demo

File: demos/models/robots/ur3_robotniq.urdf (robot description, URDF)
Before this commit: robot ur3_robotniq, 21 links, 20 joints
Joints:
- joint gripper_left_driver_joint: limit lower=0.0 upper=0.715584844444 effort=176 velocity=1.91986177778 -> lower=0.0 upper=0.872664444444 effort=60 velocity=1.91986177778

Commit message: commented line libkautham in CMakeList.txt + corrected chess demo (gripper collision model + placement of robots in problem files)

File: demos/models/robots/ur3_robotniq.urdf (robot description, URDF)
Before this commit: robot ur3_robotniq, 21 links, 20 joints
Links:
- link gripper_base: geometry collision box size=0.03 0.04 0.06; collision cylinder length=0.045 radius=0.039
- link gripper_left_coupler: geometry collision box size=0.03 0.065 0.01; visual mesh filename=robotiq/visual/coupler.dae scale=0.001 0.001 0.001
- link gripper_left_follower: geometry collision box size=0.02 0.01 0.048; visual mesh filename=robotiq/visual/follower.dae scale=0.001 0.001 0.001
- link gripper_left_pad: geometry collision box size=0.02 0.004 0.036; visual mesh filename=robotiq/visual/pad.dae scale=0.001 0.001 0.001
- link gripper_left_spring_link: geometry collision box size=0.04 0.01 0.045; visual mesh filename=robotiq/visual/spring_link.dae scale=0.001 0.001 0.001
- link gripper_right_coupler: geometry collision box size=0.03 0.065 0.01; visual mesh filename=robotiq/visual/coupler.dae scale=0.001 0.001 0.001
- link gripper_right_follower: geometry collision box size=0.02 0.01 0.048; visual mesh filename=robotiq/visual/follower.dae scale=0.001 0.001 0.001
- link gripper_right_pad: geometry collision box size=0.02 0.004 0.036; visual mesh filename=robotiq/visual/pad.dae scale=0.001 0.001 0.001
- link gripper_right_spring_link: geometry collision box size=0.04 0.01 0.045; visual mesh filename=robotiq/visual/spring_link.dae scale=0.001 0.001 0.001
- link tool0: geometry collision box size=0.01 0.01 0.001; visual box size=0.01 0.01 0.01
