Commit message: Corrected bug in urdf mesh scale definition: scale must be a vector and not an scalar

File: demos/models/obstacles/columns.urdf (robot description, URDF)
Before this commit: robot columns, 1 links, 0 joints
Links:
- link columns: geometry visual mesh filename=columns/columns.iv scale=1 1 1

File: demos/models/robots/R2D2.urdf (robot description, URDF)
Before this commit: robot R2D2, 12 links, 11 joints
Links:
- link base_link: geometry visual cylinder length=0.6 radius=0.2; visual mesh filename=R2D2/axis.iv scale=5 5 5

Commit message: Corrected examples

File: demos/models/obstacles/columns.urdf (robot description, URDF)
Before this commit: robot columns, 1 links, 0 joints
Links:
- link columns: geometry visual mesh filename=columns.iv scale=1 1 1

Commit message: Meshes in urdf must be in meters so then they must be scaled to milimeters when they are loaded

File: demos/models/obstacles/columns.urdf (robot description, URDF)
Before this commit: robot columns, 1 links, 0 joints
Links:
- link columns: geometry visual mesh filename=columns.iv scale=0.001 0.001 0.001

File: demos/models/robots/AllegroHandR.urdf (robot description, URDF)
Before this commit: robot allegro_hand_right, 21 links, 20 joints
Links:
- link Palm: geometry collision box size=0.0408 0.1130 0.095; visual mesh filename=AllegroHand/right/base_link_right.wrl scale=0.001 0.001 0.001
- link link_0.0: geometry collision box size=0.0196 0.0275 0.0164; visual mesh filename=AllegroHand/right/link_0_0.wrl scale=0.001 0.001 0.001
- link link_1.0: geometry collision box size=0.0196 0.0275 0.054; visual mesh filename=AllegroHand/right/link_1_0.wrl scale=0.001 0.001 0.001
- link link_10.0: geometry collision box size=0.0196 0.0275 0.0384; visual mesh filename=AllegroHand/right/link_2_0.wrl scale=0.001 0.001 0.001
- link link_11.0: geometry collision box size=0.0196 0.0275 0.0267; visual mesh filename=AllegroHand/right/link_3_0.wrl scale=0.001 0.001 0.001
- link link_11_0_tip: geometry collision box size=0.019 0.023 0.0365; visual mesh filename=AllegroHand/right/sensing_tip.wrl scale=0.001 0.001 0.001
- link link_12.0: geometry collision box size=0.0358 0.034 0.0455; visual mesh filename=AllegroHand/right/link_12_0_right.wrl scale=0.001 0.001 0.001
- link link_13.0: geometry collision box size=0.0196 0.0275 0.0177; visual mesh filename=AllegroHand/right/link_13_0.wrl scale=0.001 0.001 0.001
- link link_14.0: geometry collision box size=0.0196 0.0275 0.0514; visual mesh filename=AllegroHand/right/link_14_0.wrl scale=0.001 0.001 0.001
- link link_15.0: geometry collision box size=0.0196 0.0275 0.0423; visual mesh filename=AllegroHand/right/link_15_0.wrl scale=0.001 0.001 0.001
- link link_15_0_tip: geometry collision box size=0.019 0.023 0.0365; visual mesh filename=AllegroHand/right/sensing_tip.wrl scale=0.001 0.001 0.001
- link link_2.0: geometry collision box size=0.0196 0.0275 0.0384; visual mesh filename=AllegroHand/right/link_2_0.wrl scale=0.001 0.001 0.001
- link link_3.0: geometry collision box size=0.0196 0.0275 0.0267; visual mesh filename=AllegroHand/right/link_3_0.wrl scale=0.001 0.001 0.001
- link link_3_0_tip: geometry collision box size=0.019 0.023 0.0365; visual mesh filename=AllegroHand/right/sensing_tip.wrl scale=0.001 0.001 0.001
- link link_4.0: geometry collision box size=0.0196 0.0275 0.0164; visual mesh filename=AllegroHand/right/link_0_0.wrl scale=0.001 0.001 0.001
- link link_5.0: geometry collision box size=0.0196 0.0275 0.054; visual mesh filename=AllegroHand/right/link_1_0.wrl scale=0.001 0.001 0.001
- link link_6.0: geometry collision box size=0.0196 0.0275 0.0384; visual mesh filename=AllegroHand/right/link_2_0.wrl scale=0.001 0.001 0.001
- link link_7.0: geometry collision box size=0.0196 0.0275 0.0267; visual mesh filename=AllegroHand/right/link_3_0.wrl scale=0.001 0.001 0.001
- link link_7_0_tip: geometry collision box size=0.019 0.023 0.0365; visual mesh filename=AllegroHand/right/sensing_tip.wrl scale=0.001 0.001 0.001
- link link_8.0: geometry collision box size=0.0196 0.0275 0.0164; visual mesh filename=AllegroHand/right/link_0_0.wrl scale=0.001 0.001 0.001
- link link_9.0: geometry collision box size=0.0196 0.0275 0.054; visual mesh filename=AllegroHand/right/link_1_0.wrl scale=0.001 0.001 0.001

File: demos/models/robots/AllegroHandR_no_sensing.urdf (robot description, URDF)
Before this commit: robot allegro_hand_right, 21 links, 20 joints
Links:
- link Palm: geometry collision box size=0.0408 0.1130 0.095; visual mesh filename=AllegroHand/right/base_link_right.wrl scale=0.001 0.001 0.001
- link link_0.0: geometry collision box size=0.0196 0.0275 0.0164; visual mesh filename=AllegroHand/right/link_0_0.wrl scale=0.001 0.001 0.001
- link link_1.0: geometry collision box size=0.0196 0.0275 0.054; visual mesh filename=AllegroHand/right/link_1_0.wrl scale=0.001 0.001 0.001
- link link_10.0: geometry collision box size=0.0196 0.0275 0.0384; visual mesh filename=AllegroHand/right/link_2_0.wrl scale=0.001 0.001 0.001
- link link_11.0: geometry collision box size=0.0196 0.0275 0.0267; visual mesh filename=AllegroHand/right/link_3_0.wrl scale=0.001 0.001 0.001
- link link_11_0_tip: geometry collision sphere radius=0.012; visual mesh filename=AllegroHand/right/link_3_0_tip.wrl scale=0.001 0.001 0.001
- link link_12.0: geometry collision box size=0.0358 0.034 0.0455; visual mesh filename=AllegroHand/right/link_12_0_right.wrl scale=0.001 0.001 0.001
- link link_13.0: geometry collision box size=0.0196 0.0275 0.0177; visual mesh filename=AllegroHand/right/link_13_0.wrl scale=0.001 0.001 0.001
- link link_14.0: geometry collision box size=0.0196 0.0275 0.0514; visual mesh filename=AllegroHand/right/link_14_0.wrl scale=0.001 0.001 0.001
- link link_15.0: geometry collision box size=0.0196 0.0275 0.0423; visual mesh filename=AllegroHand/right/link_15_0.wrl scale=0.001 0.001 0.001
- link link_2.0: geometry collision box size=0.0196 0.0275 0.0384; visual mesh filename=AllegroHand/right/link_2_0.wrl scale=0.001 0.001 0.001
- link link_3.0: geometry collision box size=0.0196 0.0275 0.0267; visual mesh filename=AllegroHand/right/link_3_0.wrl scale=0.001 0.001 0.001
- link link_3_0_tip: geometry collision sphere radius=0.012; visual mesh filename=AllegroHand/right/link_3_0_tip.wrl scale=0.001 0.001 0.001
- link link_4.0: geometry collision box size=0.0196 0.0275 0.0164; visual mesh filename=AllegroHand/right/link_0_0.wrl scale=0.001 0.001 0.001
- link link_5.0: geometry collision box size=0.0196 0.0275 0.054; visual mesh filename=AllegroHand/right/link_1_0.wrl scale=0.001 0.001 0.001
- link link_6.0: geometry collision box size=0.0196 0.0275 0.0384; visual mesh filename=AllegroHand/right/link_2_0.wrl scale=0.001 0.001 0.001
- link link_7.0: geometry collision box size=0.0196 0.0275 0.0267; visual mesh filename=AllegroHand/right/link_3_0.wrl scale=0.001 0.001 0.001
- link link_7_0_tip: geometry collision sphere radius=0.012; visual mesh filename=AllegroHand/right/link_3_0_tip.wrl scale=0.001 0.001 0.001
- link link_8.0: geometry collision box size=0.0196 0.0275 0.0164; visual mesh filename=AllegroHand/right/link_0_0.wrl scale=0.001 0.001 0.001
- link link_9.0: geometry collision box size=0.0196 0.0275 0.054; visual mesh filename=AllegroHand/right/link_1_0.wrl scale=0.001 0.001 0.001

File: demos/models/robots/baxter.urdf (robot description, URDF)
Before this commit: robot baxter, 28 links, 27 joints
Links:
- link head: geometry collision sphere radius=0.22; collision sphere radius=0.22
- link left_gripper: geometry collision cylinder length=0.1 radius=0.0275; visual mesh filename=baxter/electric_gripper/electric_gripper_base.wrl
- link left_gripper_l_finger: geometry visual mesh filename=baxter/electric_gripper/fingers/extended_narrow.wrl
- link left_gripper_r_finger: geometry visual mesh filename=baxter/electric_gripper/fingers/extended_narrow.wrl
- link left_lower_elbow: geometry collision cylinder length=0.10 radius=0.06; visual mesh filename=baxter/lower_elbow/E1.wrl
- link left_lower_forearm: geometry collision cylinder length=0.10 radius=0.06; visual mesh filename=baxter/lower_forearm/W1.wrl
- link left_lower_shoulder: geometry collision cylinder length=0.107 radius=0.06; collision cylinder length=0.12 radius=0.06
- link left_upper_elbow: geometry collision cylinder length=0.273 radius=0.06; visual mesh filename=baxter/upper_elbow/E0.wrl
- link left_upper_forearm: geometry collision cylinder length=0.088 radius=0.06; collision cylinder length=0.272 radius=0.06
- link left_upper_shoulder: geometry collision cylinder length=0.2722 radius=0.06; visual mesh filename=baxter/upper_shoulder/S0.wrl
- link left_wrist: geometry collision cylinder length=0.165 radius=0.06; visual mesh filename=baxter/wrist/W2.wrl
- link pedestal: geometry collision mesh filename=baxter/base/pedestal_link_collision.wrl; visual mesh filename=baxter/base/PEDESTAL.wrl
- link right_gripper: geometry collision cylinder length=0.1 radius=0.0275; visual mesh filename=baxter/electric_gripper/electric_gripper_base.wrl
- link right_gripper_l_finger: geometry visual mesh filename=baxter/electric_gripper/fingers/extended_narrow.wrl
- link right_gripper_r_finger: geometry visual mesh filename=baxter/electric_gripper/fingers/extended_narrow.wrl
- link right_lower_elbow: geometry collision cylinder length=0.10 radius=0.06; visual mesh filename=baxter/lower_elbow/E1.wrl
- link right_lower_forearm: geometry collision cylinder length=0.10 radius=0.06; visual mesh filename=baxter/lower_forearm/W1.wrl
- link right_lower_shoulder: geometry collision cylinder length=0.107 radius=0.06; collision cylinder length=0.12 radius=0.06
- link right_upper_elbow: geometry collision cylinder length=0.273 radius=0.06; visual mesh filename=baxter/upper_elbow/E0.wrl
- link right_upper_forearm: geometry collision cylinder length=0.088 radius=0.06; collision cylinder length=0.272 radius=0.06
- link right_upper_shoulder: geometry collision cylinder length=0.2722 radius=0.06; visual mesh filename=baxter/upper_shoulder/S0.wrl
- link right_wrist: geometry collision cylinder length=0.165 radius=0.06; visual mesh filename=baxter/wrist/W2.wrl
- link torso: geometry collision mesh filename=baxter/torso/base_link_collision.wrl; visual mesh filename=baxter/torso/base_link.wrl

File: demos/models/robots/baxter_DAE.urdf (robot description, URDF)
Before this commit: robot baxter_DAE, 28 links, 27 joints
Links:
- link head: geometry collision sphere radius=0.22; collision sphere radius=0.22
- link left_gripper: geometry collision cylinder length=0.1 radius=0.0275; visual mesh filename=baxter_DAE/electric_gripper/electric_gripper_base.DAE
- link left_gripper_l_finger: geometry visual mesh filename=baxter_DAE/electric_gripper/fingers/extended_narrow.DAE
- link left_gripper_r_finger: geometry visual mesh filename=baxter_DAE/electric_gripper/fingers/extended_narrow.DAE
- link left_lower_elbow: geometry collision cylinder length=0.10 radius=0.06; visual mesh filename=baxter_DAE/lower_elbow/E1.DAE
- link left_lower_forearm: geometry collision cylinder length=0.10 radius=0.06; visual mesh filename=baxter_DAE/lower_forearm/W1.DAE
- link left_lower_shoulder: geometry collision cylinder length=0.107 radius=0.06; collision cylinder length=0.12 radius=0.06
- link left_upper_elbow: geometry collision cylinder length=0.273 radius=0.06; visual mesh filename=baxter_DAE/upper_elbow/E0.DAE
- link left_upper_forearm: geometry collision cylinder length=0.088 radius=0.06; collision cylinder length=0.272 radius=0.06
- link left_upper_shoulder: geometry collision cylinder length=0.2722 radius=0.06; visual mesh filename=baxter_DAE/upper_shoulder/S0.DAE
- link left_wrist: geometry collision cylinder length=0.165 radius=0.06; visual mesh filename=baxter_DAE/wrist/W2.DAE
- link pedestal: geometry collision mesh filename=baxter_DAE/base/pedestal_link_collision.DAE; visual mesh filename=baxter_DAE/base/PEDESTAL.DAE
- link right_gripper: geometry collision cylinder length=0.1 radius=0.0275; visual mesh filename=baxter_DAE/electric_gripper/electric_gripper_base.DAE
- link right_gripper_l_finger: geometry visual mesh filename=baxter_DAE/electric_gripper/fingers/extended_narrow.DAE
- link right_gripper_r_finger: geometry visual mesh filename=baxter_DAE/electric_gripper/fingers/extended_narrow.DAE
- link right_lower_elbow: geometry collision cylinder length=0.10 radius=0.06; visual mesh filename=baxter_DAE/lower_elbow/E1.DAE
- link right_lower_forearm: geometry collision cylinder length=0.10 radius=0.06; visual mesh filename=baxter_DAE/lower_forearm/W1.DAE
- link right_lower_shoulder: geometry collision cylinder length=0.107 radius=0.06; collision cylinder length=0.12 radius=0.06
- link right_upper_elbow: geometry collision cylinder length=0.273 radius=0.06; visual mesh filename=baxter_DAE/upper_elbow/E0.DAE
- link right_upper_forearm: geometry collision cylinder length=0.088 radius=0.06; collision cylinder length=0.272 radius=0.06
- link right_upper_shoulder: geometry collision cylinder length=0.2722 radius=0.06; visual mesh filename=baxter_DAE/upper_shoulder/S0.DAE
- link right_wrist: geometry collision cylinder length=0.165 radius=0.06; visual mesh filename=baxter_DAE/wrist/W2.DAE
- link torso: geometry collision mesh filename=baxter_DAE/torso/base_link_collision.DAE; visual mesh filename=baxter_DAE/torso/base_link.DAE
