Commit message: Corrected urdf models of the objects

File: demos/models/obstacles/box1.urdf (robot description, URDF)
Before this commit: robot box1, 1 links, 0 joints
Links:
- link base: geometry collision box size=0.25 0.25 0.8; visual box size=0.25 0.25 0.8

File: demos/models/obstacles/box2.urdf (robot description, URDF)
Before this commit: robot box2, 1 links, 0 joints
Links:
- link base: geometry collision box size=0.3 0.3 0.8; visual box size=0.3 0.3 0.8

File: demos/models/obstacles/box3.urdf (robot description, URDF)
Before this commit: robot box3, 1 links, 0 joints
Links:
- link base: geometry collision box size=0.3 0.3 0.8; visual box size=0.3 0.3 0.8

File: demos/models/obstacles/cubeDE1.urdf (robot description, URDF)
Before this commit: robot cubeDE, 1 links, 0 joints
Links:
- link base: geometry collision box size=0.5 0.5 0.5; visual box size=0.5 0.5 0.5

File: demos/models/obstacles/redCube1.urdf (robot description, URDF)
Before this commit: robot redcube1, 1 links, 0 joints
Links:
- link base: geometry collision box size=0.5 0.5 0.47; visual box size=0.5 0.5 0.47

File: demos/models/obstacles/redCube2.urdf (robot description, URDF)
Before this commit: robot redcube2, 1 links, 0 joints
Links:
- link base: geometry collision box size=0.5 0.5 0.47; visual box size=0.5 0.5 0.47

File: demos/models/obstacles/redCube3.urdf (robot description, URDF)
Before this commit: robot redcube3, 1 links, 0 joints
Links:
- link base: geometry collision box size=0.5 0.5 0.5; visual box size=0.5 0.5 0.5

File: demos/models/obstacles/redCube4.urdf (robot description, URDF)
Before this commit: robot redcube4, 1 links, 0 joints
Links:
- link base: geometry collision box size=0.5 0.5 0.5; visual box size=0.5 0.5 0.5
