Commit message: corrected the URDF models of the objects

File: demos/models/obstacles/cubeDE1.urdf (robot description, URDF)
Before this commit: robot cubeDE, 1 links, 0 joints
Links:
- link base: geometry collision box size=0.5 0.5 0.47; visual box size=0.5 0.5 0.47

File: demos/models/obstacles/cubeDE2.urdf (robot description, URDF)
Before this commit: robot cubeDE2, 1 links, 0 joints
Links:
- link base: geometry collision box size=0.5 0.5 0.47; visual box size=0.5 0.5 0.47

File: demos/models/obstacles/cubeDE3.urdf (robot description, URDF)
Before this commit: robot cubeDE3, 1 links, 0 joints
Links:
- link base: geometry collision box size=0.5 0.5 0.47; visual box size=0.5 0.5 0.47

File: demos/models/obstacles/cubeDE4.urdf (robot description, URDF)
Before this commit: robot cubeDE4, 1 links, 0 joints
Links:
- link base: geometry collision box size=0.5 0.5 0.47; visual box size=0.5 0.5 0.47

File: demos/models/obstacles/wall4.urdf (robot description, URDF)
Before this commit: robot wall4, 1 links, 0 joints
Links:
- link base: geometry collision box size=5.8 0.5 0.48; visual box size=5.7 0.5 0.48

File: demos/models/obstacles/wall5.urdf (robot description, URDF)
Before this commit: robot wall5, 1 links, 0 joints
Links:
- link base: geometry collision box size=1.7 0.5 0.5; visual box size=1.7 0.5 0.5

File: demos/models/obstacles/wall6.urdf (robot description, URDF)
Before this commit: robot wall6, 1 links, 0 joints
Links:
- link base: geometry collision box size=1.7 0.5 0.5; visual box size=1.7 0.5 0.5

File: demos/models/obstacles/wallb1.urdf (robot description, URDF)
Before this commit: robot wallb1, 1 links, 0 joints
Links:
- link base: geometry collision box size=9 0.5 0.5; visual box size=9 0.5 0.5

File: demos/models/obstacles/wallb2.urdf (robot description, URDF)
Before this commit: robot wallb2, 1 links, 0 joints
Links:
- link base: geometry collision box size=9 0.5 0.5; visual box size=9 0.5 0.5

File: demos/models/obstacles/wallb3.urdf (robot description, URDF)
Before this commit: robot wallb3, 1 links, 0 joints
Links:
- link base: geometry collision box size=9 0.5 0.5; visual box size=9 0.5 0.5

File: demos/models/obstacles/wallb4.urdf (robot description, URDF)
Before this commit: robot wallb4, 1 links, 0 joints
Links:
- link base: geometry collision box size=9 0.5 0.5; visual box size=9 0.5 0.5

Commit message: Corrected car demo and corrected parameters of chain planner

File: demos/models/obstacles/cubeDE1.urdf (robot description, URDF)
Before this commit: robot cubeDE, 1 links, 0 joints
Links:
- link base: mass 1 -> 0.1

File: demos/models/obstacles/cubeDE2.urdf (robot description, URDF)
Before this commit: robot cubeDE2, 1 links, 0 joints
Links:
- link base: mass 1 -> 0.1

File: demos/models/obstacles/cubeDE3.urdf (robot description, URDF)
Before this commit: robot cubeDE3, 1 links, 0 joints
Links:
- link base: mass 1 -> 0.1

File: demos/models/robots/OpenDERobots/SimpleCar.urdf (robot description, URDF)
Before this commit: robot SimpleCar, 5 links, 4 joints
Links:
- link back_left_wheel_link: geometry collision cylinder length=0.002 radius=0.002; visual cylinder length=0.002 radius=0.002
- link back_right_wheel_link: geometry collision cylinder length=0.002 radius=0.002; visual cylinder length=0.002 radius=0.002
- link base_link: mass 1.0 -> 0.2
- link front_left_wheel_link: geometry collision cylinder length=0.002 radius=0.002; visual cylinder length=0.002 radius=0.002
- link front_right_wheel_link: geometry collision cylinder length=0.002 radius=0.002; visual cylinder length=0.002 radius=0.002

Commit message: tuned parameter for physics-based towD planner

File: demos/models/obstacles/cubeDE1.urdf (robot description, URDF)
Before this commit: robot cubeDE, 1 links, 0 joints
Links:
- link base: mass 0.1 -> 0.5

File: demos/models/obstacles/cubeDE2.urdf (robot description, URDF)
Before this commit: robot cubeDE2, 1 links, 0 joints
Links:
- link base: mass 0.1 -> 0.5

File: demos/models/obstacles/cubeDE3.urdf (robot description, URDF)
Before this commit: robot cubeDE3, 1 links, 0 joints
Links:
- link base: mass 0.1 -> 0.5

File: demos/models/robots/OpenDERobots/SphereDE.urdf (robot description, URDF)
Before this commit: robot SphereDE, 1 links, 0 joints
Links:
- link base: mass 1 -> 25
