Commit message: Added collision model to the ETFA problem and modified the xml file

File: demos/models/obstacles/ETFA2016/SphereDE.urdf (robot description, URDF)
Before this commit: robot SphereDE, 1 links, 0 joints
Links:
- link base: geometry collision sphere radius=0.010; visual sphere radius=0.010

File: demos/models/obstacles/ETFA2016/cubeDE.urdf (robot description, URDF)
Before this commit: robot cubeDECoManipulatable, 1 links, 0 joints
Links:
- link base: geometry collision box size=0.02 0.02 0.02; visual box size=0.02 0.02 0.02

File: demos/models/obstacles/ETFA2016/cubeDE1.urdf (robot description, URDF)
Before this commit: robot cubeDE1, 1 links, 0 joints
Links:
- link base: geometry collision box size=0.02 0.02 0.02; visual box size=0.02 0.02 0.02

File: demos/models/obstacles/ETFA2016/cubeDE2.urdf (robot description, URDF)
Before this commit: robot cubeDE2, 1 links, 0 joints
Links:
- link base: geometry collision box size=0.02 0.02 0.02; visual box size=0.02 0.02 0.02

File: demos/models/obstacles/ETFA2016/cubeDE2IROS.urdf (robot description, URDF)
Before this commit: robot cubeDE2, 1 links, 0 joints
Links:
- link base: geometry collision box size=0.03 0.05 0.02; collision box size=0.03 0.05 0.02

File: demos/models/obstacles/ETFA2016/cubeDE3IROS.urdf (robot description, URDF)
Before this commit: robot cubeDE3, 1 links, 0 joints
Links:
- link base: geometry collision box size=0.03 0.04 0.02; visual box size=0.03 0.04 0.02

File: demos/models/obstacles/ETFA2016/cubeDE4IROS.urdf (robot description, URDF)
Before this commit: robot cubeDE4, 1 links, 0 joints
Links:
- link base: geometry collision box size=0.03 0.04 0.02; visual box size=0.03 0.04 0.02

File: demos/models/obstacles/ETFA2016/cubeDE5IROS.urdf (robot description, URDF)
Before this commit: robot cubeDE5, 1 links, 0 joints
Links:
- link base: geometry collision box size=0.03 0.04 0.02; visual box size=0.03 0.04 0.02

File: demos/models/obstacles/ETFA2016/cubeDEIROS.urdf (robot description, URDF)
Before this commit: robot cubeDE1, 1 links, 0 joints
Links:
- link base: geometry collision box size=0.03 0.04 0.02; visual box size=0.03 0.04 0.02

File: demos/models/obstacles/ETFA2016/wall10IROS.urdf (robot description, URDF)
Before this commit: robot wall10, 1 links, 0 joints
Links:
- link base: geometry collision box size=0.05 0.03 0.02; visual box size=0.05 0.03 0.02

File: demos/models/obstacles/ETFA2016/wall2IROS.urdf (robot description, URDF)
Before this commit: robot wall2, 1 links, 0 joints
Links:
- link base: geometry collision box size=0.07 0.05 0.02; visual box size=0.07 0.05 0.02

File: demos/models/obstacles/ETFA2016/wall3.urdf (robot description, URDF)
Before this commit: robot wall3, 1 links, 0 joints
Links:
- link base: geometry collision box size=0.055 0.03 0.02; visual box size=0.055 0.03 0.02

File: demos/models/obstacles/ETFA2016/wall3IROS.urdf (robot description, URDF)
Before this commit: robot wall3, 1 links, 0 joints
Links:
- link base: geometry collision box size=0.05 0.03 0.02; visual box size=0.05 0.03 0.02

File: demos/models/obstacles/ETFA2016/wall5IROS.urdf (robot description, URDF)
Before this commit: robot wall5, 1 links, 0 joints
Links:
- link base: geometry collision box size=0.07 0.05 0.02; visual box size=0.07 0.05 0.02

File: demos/models/obstacles/ETFA2016/wall6IROS.urdf (robot description, URDF)
Before this commit: robot wall6, 1 links, 0 joints
Links:
- link base: geometry collision box size=0.06 0.03 0.02; visual box size=0.06 0.03 0.02

File: demos/models/obstacles/ETFA2016/wall9IROS.urdf (robot description, URDF)
Before this commit: robot wall9, 1 links, 0 joints
Links:
- link base: geometry collision box size=0.075 0.03 0.02; visual box size=0.075 0.03 0.02

File: demos/models/obstacles/ETFA2016/wallIROS.urdf (robot description, URDF)
Before this commit: robot wall1, 1 links, 0 joints
Links:
- link base: geometry collision box size=0.15 0.03 0.02; visual box size=0.15 0.03 0.02
