Commit message: modified the code to include fcl and improve the instantiated knowledge

File: demos/models/obstacles/DEBenchmark/Plan.urdf (robot description, URDF)
Before this commit: robot Plan, 1 links, 0 joints
Links:
- link base: mass 5 -> 2

File: demos/models/obstacles/DEBenchmark/PlanDE.urdf (robot description, URDF)
Before this commit: robot Plan, 1 links, 0 joints
Links:
- link base: geometry visual box size=0.30 0.30 0.001

File: demos/models/obstacles/DEBenchmark/SphereDE.urdf (robot description, URDF)
Before this commit: robot SphereDE, 1 links, 0 joints
Links:
- link base: geometry collision sphere radius=0.010; visual sphere radius=0.010

File: demos/models/obstacles/DEBenchmark/cubeDE1.urdf (robot description, URDF)
Before this commit: robot cubeDE1, 1 links, 0 joints
Links:
- link base: geometry collision box size=0.02 0.02 0.02; visual box size=0.02 0.02 0.02

File: demos/models/obstacles/DEBenchmark/cubeDE3.urdf (robot description, URDF)
Before this commit: robot cubeDE3, 1 links, 0 joints
Links:
- link base: geometry collision box size=0.02 0.02 0.02; visual box size=0.02 0.02 0.02

File: demos/models/obstacles/ETFA2016/wall8IROS.urdf (robot description, URDF)
Before this commit: robot wall8, 1 links, 0 joints
Links:
- link base: geometry collision box size=0.12 0.03 0.02; visual box size=0.12 0.03 0.02

File: demos/models/obstacles/IROS/PlanerChain.urdf (robot description, URDF)
Before this commit: robot Chain, 4 links, 3 joints
Links:
- link gripper: geometry collision box size=0.002 0.006 0.002; visual box size=0.002 0.006 0.002
- link link1: geometry collision box size=0.01 0.01 0.1; visual box size=0.01 0.01 0.1
- link link2: geometry collision box size=0.01 0.01 0.1; visual box size=0.01 0.01 0.1
Joints:
- joint joint1: origin xyz=0 0 0.01 -> xyz=0 0 0.02
- joint joint2: origin xyz=0 0 0.2 -> xyz=0 0 0.1
- joint joint3: origin xyz=0 0 0.2 -> xyz=0 0 0.1
