Commit message: merge different robot models (car, chain ..)

File: demos/models/obstacles/DEBenchmark/Car.urdf (robot description, URDF)
Before this commit: robot SimpleCar, 5 links, 4 joints
Links:
- link back_left_wheel_link: mass 0.01 -> 1
- link back_right_wheel_link: mass 0.01 -> 1
- link base_link: mass 0.2 -> 2
- link front_left_wheel_link: mass 0.01 -> 1
- link front_right_wheel_link: mass 0.01 -> 1

File: demos/models/obstacles/DEBenchmark/Plan.urdf (robot description, URDF)
Before this commit: robot Plan, 1 links, 0 joints
Links:
- link base: geometry collision box size=1 1 0.002; visual box size=1 1 0.002

File: demos/models/obstacles/DEBenchmark/cubeDE2.urdf (robot description, URDF)
Before this commit: robot cubeDE2, 1 links, 0 joints
Links:
- link base: geometry collision box size=0.02 0.02 0.02; visual box size=0.02 0.02 0.02

File: demos/models/obstacles/DEBenchmark/wall4.urdf (robot description, URDF)
Before this commit: robot wall4, 1 links, 0 joints
Links:
- link base: geometry collision box size=0.2 0.03 0.02; visual box size=0.2 0.03 0.02
