Commit message: updated demos

File: demos/models/obstacles/DEBenchmark/PlanDE.urdf (robot description, URDF)
Before this commit: robot Plan, 1 links, 0 joints
Links:
- link base: geometry collision box size=0.15 0.03 0.02; visual box size=0.30 0.30 0.001

File: demos/models/obstacles/DEBenchmark/cubeDE.urdf (robot description, URDF)
Before this commit: robot cubeDECoManipulatable, 1 links, 0 joints
Links:
- link base: geometry collision box size=0.02 0.02 0.02; visual box size=0.02 0.02 0.02

File: demos/models/obstacles/DEBenchmark/wall1.urdf (robot description, URDF)
Before this commit: robot wall1, 1 links, 0 joints
Links:
- link base: geometry collision box size=0.15 0.03 0.02; visual box size=0.15 0.03 0.02

File: demos/models/obstacles/DEBenchmark/wall2.urdf (robot description, URDF)
Before this commit: robot wall2, 1 links, 0 joints
Links:
- link base: geometry collision box size=0.2 0.03 0.02; visual box size=0.2 0.03 0.02

File: demos/models/obstacles/DEBenchmark/wall3.urdf (robot description, URDF)
Before this commit: robot wall3, 1 links, 0 joints
Links:
- link base: geometry collision box size=0.055 0.03 0.02; visual box size=0.055 0.03 0.02
