Commit message: added function to visulize the triangular mesh in drawstuff

File: demos/models/obstacles/DSTest/twoLink.urdf (robot description, URDF)
Before this commit: robot Chain, 4 links, 3 joints
Joints:
- joint joint1: origin xyz=0 0 0.0031 -> xyz=0 0 0.003
- joint joint2: limit lower=-2.40 upper=2.40 effort=300 velocity=0.1 -> lower=-1.50 upper=1.50 effort=300 velocity=0.1
