Commit message: completed chess demo

File: demos/models/obstacles/chess/kingB.urdf (robot description, URDF)
Before this commit: robot pawnW1, 1 links, 0 joints
Links:
- link base: geometry collision box size=0.03 0.03 0.08; visual mesh filename=visual/kingB.dae scale=0.6 0.6 1.6

File: demos/models/obstacles/chess/kingW.urdf (robot description, URDF)
Before this commit: robot cheassboard, 1 links, 0 joints
Links:
- link base: geometry collision box size=0.03 0.03 0.08; visual mesh filename=visual/kingW.dae scale=0.6 0.6 1.6

File: demos/models/obstacles/chess/knightW2.urdf (robot description, URDF)
Before this commit: robot cheassboard, 1 links, 0 joints
Links:
- link base: geometry collision box size=0.03 0.03 0.06; visual mesh filename=visual/knightW2.dae scale=0.6 0.6 1.2

File: demos/models/obstacles/chess/pawnW2.urdf (robot description, URDF)
Before this commit: robot pawnW1, 1 links, 0 joints
Links:
- link base: geometry collision box size=0.03 0.03 0.04; visual mesh filename=visual/pawnW2.dae scale=0.6 0.6 0.8

File: demos/models/obstacles/chess/queenB.urdf (robot description, URDF)
Before this commit: robot pawnW1, 1 links, 0 joints
Links:
- link base: geometry collision box size=0.03 0.03 0.08; visual mesh filename=visual/queenB.dae scale=0.6 0.6 1.6

File: demos/models/obstacles/chess/queenW.urdf (robot description, URDF)
Before this commit: robot pawnW1, 1 links, 0 joints
Links:
- link base: geometry collision box size=0.03 0.03 0.08; visual mesh filename=visual/queenW.dae scale=0.6 0.6 1.6

File: demos/models/robots/ur3_robotniq.urdf (robot description, URDF)
Before this commit: robot ur3_robotniq, 7 links, 6 joints
Joints:
- joint shoulder_lift_joint: limit lower=-6.28318530718 upper=6.28318530718 effort=330.0 velocity=2.16 -> lower=-3.141592654 upper=3.141592654 effort=330.0 velocity=2.16
- joint shoulder_pan_joint: limit lower=-6.28318530718 upper=6.28318530718 effort=330.0 velocity=2.16 -> lower=-3.141592654 upper=3.141592654 effort=330.0 velocity=2.16
- joint wrist_1_joint: limit lower=-6.28318530718 upper=6.28318530718 effort=54.0 velocity=3.2 -> lower=-3.141592654 upper=3.141592654 effort=54.0 velocity=3.2
- joint wrist_2_joint: limit lower=-6.28318530718 upper=6.28318530718 effort=54.0 velocity=3.2 -> lower=-3.141592654 upper=3.141592654 effort=54.0 velocity=3.2
- joint wrist_3_joint: limit lower=-6.28318530718 upper=6.28318530718 effort=54.0 velocity=3.2 -> lower=-3.141592654 upper=3.141592654 effort=54.0 velocity=3.2
