Commit message: corrected dimensions in chess demo

File: demos/models/obstacles/chess/chessboard.urdf (robot description, URDF)
Before this commit: robot cheassboard, 1 links, 0 joints
Links:
- link base: geometry collision box size=0.46 0.46 0.04; visual mesh filename=visual/chessboard.dae scale=9.2 9.2 0.8

Commit message: cleaned comments. Corrected chess example - objects have all base_link

File: demos/models/obstacles/chess/chessboard.urdf (robot description, URDF)
Before this commit: robot cheassboard, 1 links, 0 joints
Links:
- removed link base
- added link base_link; collision box size=0.46 0.46 0.04; visual mesh filename=visual/chessboard.dae scale=9.2 9.2 0.8

File: demos/models/obstacles/chess/horseB1.urdf (robot description, URDF)
Before this commit: robot horseB1, 1 links, 0 joints
Links:
- removed link base
- added link base_link; collision box size=0.03 0.03 0.06; visual mesh filename=visual/horseB1.dae scale=0.6 0.6 1.2

File: demos/models/obstacles/chess/horseB2.urdf (robot description, URDF)
Before this commit: robot horseB2, 1 links, 0 joints
Links:
- removed link base
- added link base_link; collision box size=0.03 0.03 0.06; visual mesh filename=visual/horseB2.dae scale=0.6 0.6 1.2

File: demos/models/obstacles/chess/horseW1.urdf (robot description, URDF)
Before this commit: robot horseW1, 1 links, 0 joints
Links:
- removed link base
- added link base_link; collision box size=0.03 0.03 0.06; visual mesh filename=visual/horseW1.dae scale=0.6 0.6 1.2

File: demos/models/obstacles/chess/horseW2.urdf (robot description, URDF)
Before this commit: robot horseW2, 1 links, 0 joints
Links:
- removed link base
- added link base_link; collision box size=0.03 0.03 0.06; visual mesh filename=visual/horseW2.dae scale=0.6 0.6 1.2

File: demos/models/obstacles/chess/kingB.urdf (robot description, URDF)
Before this commit: robot kingB, 1 links, 0 joints
Links:
- removed link base
- added link base_link; collision box size=0.03 0.03 0.08; visual mesh filename=visual/kingB.dae scale=0.6 0.6 1.6

File: demos/models/obstacles/chess/kingW.urdf (robot description, URDF)
Before this commit: robot kingW, 1 links, 0 joints
Links:
- removed link base
- added link base_link; collision box size=0.03 0.03 0.08; visual mesh filename=visual/kingW.dae scale=0.6 0.6 1.6

File: demos/models/obstacles/chess/knightB1.urdf (robot description, URDF)
Before this commit: robot knightB1, 1 links, 0 joints
Links:
- removed link base
- added link base_link; collision box size=0.03 0.03 0.06; visual mesh filename=visual/knightB1.dae scale=0.6 0.6 1.2

File: demos/models/obstacles/chess/knightB2.urdf (robot description, URDF)
Before this commit: robot knightB2, 1 links, 0 joints
Links:
- removed link base
- added link base_link; collision box size=0.03 0.03 0.06; visual mesh filename=visual/knightB2.dae scale=0.6 0.6 1.2

File: demos/models/obstacles/chess/knightW1.urdf (robot description, URDF)
Before this commit: robot knightW1, 1 links, 0 joints
Links:
- removed link base
- added link base_link; collision box size=0.03 0.03 0.06; visual mesh filename=visual/knightW1.dae scale=0.6 0.6 1.2

File: demos/models/obstacles/chess/knightW2.urdf (robot description, URDF)
Before this commit: robot knightW2, 1 links, 0 joints
Links:
- removed link base
- added link base_link; collision box size=0.03 0.03 0.06; visual mesh filename=visual/knightW2.dae scale=0.6 0.6 1.2

File: demos/models/obstacles/chess/pawnB1.urdf (robot description, URDF)
Before this commit: robot pawnB1, 1 links, 0 joints
Links:
- removed link base
- added link base_link; collision box size=0.03 0.03 0.04; visual mesh filename=visual/pawnB1.dae scale=0.6 0.6 0.8

File: demos/models/obstacles/chess/pawnB2.urdf (robot description, URDF)
Before this commit: robot pawnB2, 1 links, 0 joints
Links:
- removed link base
- added link base_link; collision box size=0.03 0.03 0.04; visual mesh filename=visual/pawnB2.dae scale=0.6 0.6 0.8

File: demos/models/obstacles/chess/pawnB3.urdf (robot description, URDF)
Before this commit: robot pawnB3, 1 links, 0 joints
Links:
- removed link base
- added link base_link; collision box size=0.03 0.03 0.04; visual mesh filename=visual/pawnB3.dae scale=0.6 0.6 0.8

File: demos/models/obstacles/chess/pawnB4.urdf (robot description, URDF)
Before this commit: robot pawnB4, 1 links, 0 joints
Links:
- removed link base
- added link base_link; collision box size=0.03 0.03 0.04; visual mesh filename=visual/pawnB4.dae scale=0.6 0.6 0.8

File: demos/models/obstacles/chess/pawnB5.urdf (robot description, URDF)
Before this commit: robot pawnB5, 1 links, 0 joints
Links:
- removed link base
- added link base_link; collision box size=0.03 0.03 0.04; visual mesh filename=visual/pawnB5.dae scale=0.6 0.6 0.8

File: demos/models/obstacles/chess/pawnB6.urdf (robot description, URDF)
Before this commit: robot pawnB6, 1 links, 0 joints
Links:
- removed link base
- added link base_link; collision box size=0.03 0.03 0.04; visual mesh filename=visual/pawnB6.dae scale=0.6 0.6 0.8

File: demos/models/obstacles/chess/pawnB7.urdf (robot description, URDF)
Before this commit: robot pawnB7, 1 links, 0 joints
Links:
- removed link base
- added link base_link; collision box size=0.03 0.03 0.04; visual mesh filename=visual/pawnB7.dae scale=0.6 0.6 0.8

File: demos/models/obstacles/chess/pawnB8.urdf (robot description, URDF)
Before this commit: robot pawnB8, 1 links, 0 joints
Links:
- removed link base
- added link base_link; collision box size=0.03 0.03 0.04; visual mesh filename=visual/pawnB8.dae scale=0.6 0.6 0.8

File: demos/models/obstacles/chess/pawnW1.urdf (robot description, URDF)
Before this commit: robot pawnW1, 1 links, 0 joints
Links:
- removed link base
- added link base_link; collision box size=0.03 0.03 0.04; visual mesh filename=visual/pawnW1.dae scale=0.6 0.6 0.8
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
Commit message: chess ok. tiago in process

File: demos/models/obstacles/chess/chessboard.urdf (robot description, URDF)
Before this commit: robot cheassboard, 1 links, 0 joints
Links:
- removed link base_link
- added link base; collision box size=0.46 0.46 0.04; visual mesh filename=visual/chessboard.dae scale=9.2 9.2 0.8

File: demos/models/obstacles/chess/horseB1.urdf (robot description, URDF)
Before this commit: robot horseB1, 1 links, 0 joints
Links:
- removed link base_link
- added link base; collision box size=0.03 0.03 0.06; visual mesh filename=visual/horseB1.dae scale=0.6 0.6 1.2

File: demos/models/obstacles/chess/horseB2.urdf (robot description, URDF)
Before this commit: robot horseB2, 1 links, 0 joints
Links:
- removed link base_link
- added link base; collision box size=0.03 0.03 0.06; visual mesh filename=visual/horseB2.dae scale=0.6 0.6 1.2

File: demos/models/obstacles/chess/horseW1.urdf (robot description, URDF)
Before this commit: robot horseW1, 1 links, 0 joints
Links:
- removed link base_link
- added link base; collision box size=0.03 0.03 0.06; visual mesh filename=visual/horseW1.dae scale=0.6 0.6 1.2

File: demos/models/obstacles/chess/horseW2.urdf (robot description, URDF)
Before this commit: robot horseW2, 1 links, 0 joints
Links:
- removed link base_link
- added link base; collision box size=0.03 0.03 0.06; visual mesh filename=visual/horseW2.dae scale=0.6 0.6 1.2

File: demos/models/obstacles/chess/kingB.urdf (robot description, URDF)
Before this commit: robot kingB, 1 links, 0 joints
Links:
- removed link base_link
- added link base; collision box size=0.03 0.03 0.08; visual mesh filename=visual/kingB.dae scale=0.6 0.6 1.6

File: demos/models/obstacles/chess/kingW.urdf (robot description, URDF)
Before this commit: robot kingW, 1 links, 0 joints
Links:
- removed link base_link
- added link base; collision box size=0.03 0.03 0.08; visual mesh filename=visual/kingW.dae scale=0.6 0.6 1.6

File: demos/models/obstacles/chess/knightB1.urdf (robot description, URDF)
Before this commit: robot knightB1, 1 links, 0 joints
Links:
- removed link base_link
- added link base; collision box size=0.03 0.03 0.06; visual mesh filename=visual/knightB1.dae scale=0.6 0.6 1.2

File: demos/models/obstacles/chess/knightB2.urdf (robot description, URDF)
Before this commit: robot knightB2, 1 links, 0 joints
Links:
- removed link base_link
- added link base; collision box size=0.03 0.03 0.06; visual mesh filename=visual/knightB2.dae scale=0.6 0.6 1.2

File: demos/models/obstacles/chess/knightW1.urdf (robot description, URDF)
Before this commit: robot knightW1, 1 links, 0 joints
Links:
- removed link base_link
- added link base; collision box size=0.03 0.03 0.06; visual mesh filename=visual/knightW1.dae scale=0.6 0.6 1.2

File: demos/models/obstacles/chess/knightW2.urdf (robot description, URDF)
Before this commit: robot knightW2, 1 links, 0 joints
Links:
- removed link base_link
- added link base; collision box size=0.03 0.03 0.06; visual mesh filename=visual/knightW2.dae scale=0.6 0.6 1.2

File: demos/models/obstacles/chess/pawnB1.urdf (robot description, URDF)
Before this commit: robot pawnB1, 1 links, 0 joints
Links:
- removed link base_link
- added link base; collision box size=0.03 0.03 0.04; visual mesh filename=visual/pawnB1.dae scale=0.6 0.6 0.8

File: demos/models/obstacles/chess/pawnB2.urdf (robot description, URDF)
Before this commit: robot pawnB2, 1 links, 0 joints
Links:
- removed link base_link
- added link base; collision box size=0.03 0.03 0.04; visual mesh filename=visual/pawnB2.dae scale=0.6 0.6 0.8

File: demos/models/obstacles/chess/pawnB3.urdf (robot description, URDF)
Before this commit: robot pawnB3, 1 links, 0 joints
Links:
- removed link base_link
- added link base; collision box size=0.03 0.03 0.04; visual mesh filename=visual/pawnB3.dae scale=0.6 0.6 0.8

File: demos/models/obstacles/chess/pawnB4.urdf (robot description, URDF)
Before this commit: robot pawnB4, 1 links, 0 joints
Links:
- removed link base_link
- added link base; collision box size=0.03 0.03 0.04; visual mesh filename=visual/pawnB4.dae scale=0.6 0.6 0.8

File: demos/models/obstacles/chess/pawnB5.urdf (robot description, URDF)
Before this commit: robot pawnB5, 1 links, 0 joints
Links:
- removed link base_link
- added link base; collision box size=0.03 0.03 0.04; visual mesh filename=visual/pawnB5.dae scale=0.6 0.6 0.8

File: demos/models/obstacles/chess/pawnB6.urdf (robot description, URDF)
Before this commit: robot pawnB6, 1 links, 0 joints
Links:
- removed link base_link
- added link base; collision box size=0.03 0.03 0.04; visual mesh filename=visual/pawnB6.dae scale=0.6 0.6 0.8

File: demos/models/obstacles/chess/pawnB7.urdf (robot description, URDF)
Before this commit: robot pawnB7, 1 links, 0 joints
Links:
- removed link base_link
- added link base; collision box size=0.03 0.03 0.04; visual mesh filename=visual/pawnB7.dae scale=0.6 0.6 0.8

File: demos/models/obstacles/chess/pawnB8.urdf (robot description, URDF)
Before this commit: robot pawnB8, 1 links, 0 joints
Links:
- removed link base_link
- added link base; collision box size=0.03 0.03 0.04; visual mesh filename=visual/pawnB8.dae scale=0.6 0.6 0.8

File: demos/models/obstacles/chess/pawnW1.urdf (robot description, URDF)
Before this commit: robot pawnW1, 1 links, 0 joints
Links:
- removed link base_link
- added link base; collision box size=0.03 0.03 0.04; visual mesh filename=visual/pawnW1.dae scale=0.6 0.6 0.8
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