Commit message: corrected collision issue

File: demos/models/obstacles/chess/flat_chessboard.urdf (robot description, URDF)
Before this commit: robot flat_chessboard, 1 links, 0 joints
Links:
- link base: geometry collision box size=0.65 0.6 0.004; visual box size=0.70 0.65 0.0039

Commit message: chess demo: split flat chessboard into support+chessboard

File: demos/models/obstacles/chess/flat_chessboard.urdf (robot description, URDF)
Before this commit: robot flat_chessboard, 1 links, 0 joints
Links:
- link base: geometry collision box size=0.594 0.42 0.004; visual mesh filename=visual/flat_chessboard.dae scale=11.88 8.4 0.08
