Commit message: improved kithchen model

File: demos/models/obstacles/kitchen/kitchen.urdf (robot description, URDF)
Before this commit: robot bottle8, 1 links, 0 joints
Links:
- link base: geometry collision mesh filename=kitchen_simple/kitchen_simple.dae scale=0.0254 0.0254 0.0254; visual mesh filename=kitchen_simple/kitchen_simple.dae scale=0.0254 0.0254 0.0254
