Commit message: modified models for tiago. Includes xacro files that use the find package macro to find ethe geometries; to be used by the tiago_arm_kinematics package to find IK. Left cases work find in kautham but the IK not available

File: demos/models/obstacles/kitchen/glass.urdf (robot description, URDF)
Before this commit: robot glass, 1 links, 0 joints
Links:
- link base: geometry collision mesh filename=Glass.dae scale=0.0254 0.0254 0.0254; visual mesh filename=Glass.dae scale=0.0254 0.0254 0.0254
