Commit message: rviz visualization correct with tiago-kitchen

File: demos/models/obstacles/kitchen/can.urdf (robot description, URDF)
Before this commit: robot can, 1 links, 0 joints
Links:
- link base: geometry collision mesh filename=can/cokecan.dae scale=0.0254 0.0254 0.0254; visual mesh filename=can/cokecan2.dae scale=0.0254 0.0254 0.0254

Commit message: modified collision model of can object

File: demos/models/obstacles/kitchen/can.urdf (robot description, URDF)
Before this commit: robot can, 1 links, 0 joints
Links:
- link base: geometry collision cylinder length=0.11 radius=0.030; visual mesh filename=can/cokecan2.dae scale=0.0254 0.0254 0.0254
