Commit message: all demos revised according to use only urdf format

File: demos/models/obstacles/TMP/cube-big.urdf (robot description, URDF)
Before this commit: robot box8, 1 links, 0 joints
Links:
- link base: mass 1 -> None; geometry collision mesh filename=cube-big.wrl scale=1.0 1.0 1.0; visual mesh filename=cube-big.wrl scale=1.0 1.0 1.0

File: demos/models/obstacles/ode-objects/box1.urdf (robot description, URDF)
Before this commit: robot box1, 1 links, 0 joints
Links:
- link base: mass 0.04 -> 0.2; geometry collision box size=0.25 0.25 0.8; visual box size=0.25 0.25 0.8

File: demos/models/obstacles/ode-objects/box2.urdf (robot description, URDF)
Before this commit: robot box2, 1 links, 0 joints
Links:
- link base: mass 0.05 -> 0.4; geometry collision box size=0.3 0.3 0.8; visual box size=0.3 0.3 0.8

File: demos/models/obstacles/ode-objects/box3.urdf (robot description, URDF)
Before this commit: robot box3, 1 links, 0 joints
Links:
- link base: mass 0.05 -> 0.4; geometry collision box size=0.3 0.3 0.8; visual box size=0.3 0.3 0.8

File: demos/models/obstacles/ode-objects/box4.urdf (robot description, URDF)
Before this commit: robot box4, 1 links, 0 joints
Links:
- link base: mass 0.05 -> 0.1; geometry collision box size=0.007 0.007 0.015; visual box size=0.007 0.007 0.015

File: demos/models/robots/UR5_AllegroHandL_cylinder.urdf (robot description, URDF)
Before this commit: robot UR5_AllegroHandL, 30 links, 29 joints
Links:
- link Cylinder: geometry visual mesh filename=AllegroHand/objects/cylinder.wrl scale=0.001 0.001 0.001

File: demos/models/robots/UR5_AllegroHandR_cylinder.urdf (robot description, URDF)
Before this commit: robot UR5_AllegroHandR, 30 links, 29 joints
Links:
- link Can: geometry visual mesh filename=AllegroHand/objects/can.wrl

File: demos/models/robots/UR5_AllegroHandR_water.urdf (robot description, URDF)
Before this commit: robot UR5_AllegroHandR, 30 links, 29 joints
Links:
- link Can: geometry visual mesh filename=AllegroHand/objects/can.wrl
