Commit message: corrected tiago urdf model to set torso and fingers not fixed

File: demos/models/robots/tiago/tiago_with_gripper.urdf (robot description, URDF)
Before this commit: robot tiago, 17 links, 16 joints
Joints:
- joint arm_6_joint: type fixed -> revolute
- joint arm_7_joint: type fixed -> revolute
- joint torso_lift_joint: type fixed -> prismatic

Commit message: working on Tiago. Using dae files for visualization instead of stl

File: demos/models/robots/tiago/tiago_with_gripper.urdf (robot description, URDF)
Before this commit: robot tiago, 17 links, 16 joints
Links:
- link arm_1_link: geometry collision mesh filename=tiago/meshes/arm/arm_1_collision.dae scale=1 1 1; visual mesh filename=tiago/meshes/arm/arm_1_collision.dae scale=1 1 1
- link arm_2_link: geometry collision mesh filename=tiago/meshes/arm/arm_2_collision.dae scale=1 1 1; visual mesh filename=tiago/meshes/arm/arm_2_collision.dae scale=1 1 1
- link arm_3_link: geometry collision mesh filename=tiago/meshes/arm/arm_3_collision.dae scale=1 1 1; visual mesh filename=tiago/meshes/arm/arm_3_collision.dae scale=1 1 1
- link arm_4_link: geometry collision mesh filename=tiago/meshes/arm/arm_4_collision.dae scale=1 1 1; visual mesh filename=tiago/meshes/arm/arm_4_collision.dae scale=1 1 1
- link arm_5_link: geometry collision mesh filename=tiago/meshes/arm/arm_5_collision.dae scale=1 1 1; visual mesh filename=tiago/meshes/arm/arm_5_collision.dae scale=1 1 1
- link arm_6_link: geometry collision mesh filename=tiago/meshes/arm/arm_6_collision.dae scale=1 1 1; visual mesh filename=tiago/meshes/arm/arm_6_collision.dae scale=1 1 1
- link base_link: geometry collision mesh filename=tiago/meshes/base/base_collision.dae; visual mesh filename=tiago/meshes/base/base_collision.dae
- link head_1_link: geometry collision mesh filename=tiago/meshes/head/head_1_collision.dae scale=1 1 1; visual mesh filename=tiago/meshes/head/head_1_collision.dae scale=1 1 1
- link head_2_link: geometry collision mesh filename=tiago/meshes/head/head_2_collision.dae scale=1 1 1; visual mesh filename=tiago/meshes/head/head_2_collision.dae scale=1 1 1
- link torso_fixed_link: geometry collision box size=0.25 0.25 0.1; collision box size=0.4 0.25 0.04
- link torso_lift_link: geometry collision mesh filename=tiago/meshes/torso/torso_lift_collision.dae scale=1 1 1; visual mesh filename=tiago/meshes/torso/torso_lift_collision.dae scale=1 1 1
- link wheel_left_link: geometry collision cylinder length=0.04 radius=0.0985; visual cylinder length=0.04 radius=0.0985
- link wheel_right_link: geometry collision cylinder length=0.04 radius=0.0985; visual cylinder length=0.04 radius=0.0985

Commit message: debugging

File: demos/models/robots/tiago/tiago_with_gripper.urdf (robot description, URDF)
Before this commit: robot tiago, 17 links, 16 joints
Links:
- added link arm_tool_link, mass 0.1; collision cylinder length=0.005 radius=0.005; visual cylinder length=0.005 radius=0.005
Joints:
- added joint arm_tool_joint: type fixed, parent arm_7_link, child arm_tool_link, origin xyz=0 0 0.046 rpy=1.57079632679 -1.57079632679 3.1415
