Commit message: Nadal commit: Added MADAR with only the arm right (DEBUG).

File: demos/models/robots/MADAR/madar_arm_right.urdf (robot description, URDF)
Before this commit: robot madar_arm_right, 11 links, 10 joints
Links:
- removed link wheel_1_link
- removed link wheel_2_link
- removed link wheel_3_link
Joints:
- removed joint motor_1
- removed joint motor_2
- removed joint motor_3
- joint right_base_link: limit (none) -> lower=-0.01 upper=0.01 effort=0.0 velocity=0.0
